File: MSX_IDC_Interface.kicad_pcb (KiCad board)
At the start: 2 copper layers, 103 x 66 mm, 27 parts, among them J1 DE1 GPIO, J2 Conn_01x03_Male, J3 Conn_01x03_Male, J4 Conn_01x03_Male, J5 Conn_01x03_Male, J6 Conn_01x03_Male, J7 Conn_01x03_Male, U1 74LVC245A, U2 74LVC245A, U3 74LVC245A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

Commit message: Version 1.0 with fabrication files
Parts:
- added G***: LOGO, LOGO, B.Cu at (81.7, 30.8)
- added G***: LOGO, LOGO, B.Cu at (107.2, 66.0)
- added G***: LOGO, LOGO, B.Cu at (99.6, 51.8)
- added G***: LOGO, LOGO, B.Cu at (110.7, 34.0)

Commit message: Repositioned background silk and removed unwanted G** in the galaga silk. Continue being Verison 1.0
Parts:
- moved G*** 15.7 mm to (66.0, 32.0)
- moved G*** 1.02 mm to (107.2, 67.1)
Changed lines of the file:
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@@
   )
   (footprint "LOGO" (layer "B.Cu")
-    (at 81.672214 30.779377 180)
+    (at 66.04 32.004 180)
     (attr board_only exclude_from_pos_files exclude_from_bom)
-    (fp_text reference "G***" (at 0 0) (layer "B.SilkS")
+    (fp_text reference "G***" (at 0 0) (layer "B.SilkS") hide
       (effects (font (size 1.524 1.524) (thickness 0.3)) (justify mirror))
     )
@@
   )
   (footprint "LOGO" (layer "B.Cu")
-    (at 107.188 66.04 180)
+    (at 107.188 67.056 180)
     (attr board_only exclude_from_pos_files exclude_from_bom)
     (fp_text reference "G***" (at 0 0) (layer "B.SilkS") hide

Commit message: Fixed missing 3v input
Connections:
- J1 pad 29: unconnected-(J1-Pad29) -> +3.3V
Routing:
- net +3.3V: track 237.9 -> 256.4 mm
- net (no net): vias 0 -> 1
