File: Hardware Interface/DE0_Addon_Board/DE0_Addon_Board.kicad_sch (KiCad schematic)
At the start: 5 parts, among them J1 Conn_02x20_Odd_Even, J2 Conn_01x05_Male, U1 IS61WV25616EDBLL

Commit message: Added 2nd IDC connector in paralell with the SRAM
Parts:
- removed J2: Conn_01x05_Male, Connector_PinHeader_2.54mm:PinHeader_1x05_P2.54mm_Vertical, symbol Connector:Conn_01x05_Male
- added J2: Conn_01x02_Male, Jumper:SolderJumper-2_P1.3mm_Open_Pad1.0x1.5mm, symbol Jumper:SolderJumper_2_Open
- added J3: Conn_02x20_Odd_Even, Connector_PinHeader_2.54mm:PinHeader_2x20_P2.54mm_Vertical, symbol Connector_Generic:Conn_02x20_Odd_Even
Connections:
- net +3.3V: now also J3.29 (Pin_29)
- net A0: now also J3.2 (Pin_2)
- net A1: now also J3.4 (Pin_4)
- net A10: now also J3.27 (Pin_27)
- net A11: now also J3.28 (Pin_28)
- net A12: now also J3.25 (Pin_25)
- net A13: now also J3.26 (Pin_26)
- net A14: now also J3.23 (Pin_23)
- net A15: now also J3.18 (Pin_18)
- net A16: now also J3.15 (Pin_15)
- net A17: now also J3.16 (Pin_16)
- net A2: now also J3.5 (Pin_5)
- net A3: now also J3.6 (Pin_6)
- net A4: now also J3.7 (Pin_7)
- net A5: now also J3.35 (Pin_35)
- net A6: now also J3.38 (Pin_38)
- net A7: now also J3.37 (Pin_37)
- net A8: now also J3.40 (Pin_40)
- net A9: now also J3.39 (Pin_39)
- net CE_n: now also J2.2 (B), J3.8 (Pin_8); no longer U1.6 (~{CE})
- net D0: now also J3.9 (Pin_9)
- net D1: now also J3.10 (Pin_10)
- net D10: now also J3.14 (Pin_14)
- net D11: now also J3.13 (Pin_13)
- net D12: now also J3.32 (Pin_32)
- net D13: now also J3.31 (Pin_31)
- net D14: now also J3.34 (Pin_34)
- net D15: now also J3.33 (Pin_33)
- net GNDREF: now also J3.12 (Pin_12), J3.30 (Pin_30)
- net LB_n: now also J3.19 (Pin_19)
- net OE_n: now also J3.17 (Pin_17)
- net P1: now also J3.1 (Pin_1)
- net P21: now also J3.21 (Pin_21)
- net P22: now also J3.22 (Pin_22)
- net P24: now also J3.24 (Pin_24)
- net P3: now also J3.3 (Pin_3)
- net UB_n: now also J3.20 (Pin_20)
- net WE_n: now also J3.36 (Pin_36)
- new net MEM_CE_n: J2.1 (A), U1.6 (~{CE})
- no-connect marks 1 -> 2
Other:
- moved on the sheet: C1, C2
