File: Hardware Interface/MSX_FPGA_Hat.kicad_pcb (KiCad board)
At the start: 2 copper layers, 99.9 x 64 mm, 41 parts, among them J1 Conn_01x03_Female, J2 SND, J3 AudioJack3, J4 /CS12, Q1 2N3904, Q2 2N3904, SW1 RESET, U1 74LVC245, U2 74LVC245, U3 74LVC245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

Commit message: V2.01
Parts:
- added J5: RFSH_CS2, Jumper:SolderJumper-3_P1.3mm_Open_RoundedPad1.0x1.5mm, F.Cu at (127.9, 46.7)
- J2: value SND -> Soundin
- moved CONN1 0.18 mm to (99.1, 53.1)
Connections:
- U4 pad 16: /C_CS2_RFSH -> /C_RFSH
- U5 pad 14: /C_CS2_RFSH -> /C_CS2
Routing:
- net /C_CS2_RFSH: track 47.8 -> 22.7 mm
- net /C_CS2: track 0.00 -> 22.3 mm, vias 0 -> 1
- net /C_RFSH: track 0.00 -> 4.92 mm
- net GNDREF: track 468.0 -> 463.8 mm
- net Vcc: track 160.7 -> 159.3 mm

Commit message: Master is currentl under development and tests for v2.0
Parts:
- removed J5: RFSH_CS2, Jumper:SolderJumper-3_P1.3mm_Open_RoundedPad1.0x1.5mm
Connections:
- IDC1 pad 10: /C_U4_OE -> /C_CS2
- IDC1 pad 6: /C_CS2_RFSH -> /C_RFSH
- U4 pad 19: /C_U4_OE -> GNDREF
Routing:
- net /C_CS2: track 22.3 -> 50.0 mm, vias 1 -> 3
- net /C_CS2_RFSH: track 22.7 -> 0.00 mm
- net /C_RFSH: track 4.92 -> 27.2 mm
- net GNDREF: track 463.8 -> 485.1 mm
- net /C_U4_OE: track 20.5 -> 0.00 mm
- net /SLTSL: track 46.8 -> 46.1 mm
