File: Hardware Interface/MSX_FPGA_Hat.kicad_sch (KiCad schematic)
At the start: 40 parts, among them J1 Conn_01x03_Female, J2 Soundin, J3 AudioJack3, J4 /CS12, Q1 2N3904, Q2 2N3904, SW1 RESET, U1 74LVC245, U2 74LVC245, U3 74LVC245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

Commit message: v2.0 has a bug - added a info in the schematic
Other:
- note added: "v2.0 Bug: CS2 & RFSH sharing same pin but OE is grounded. RFSH should not be wired (soldered) in U4 to avoid issues."
Changed lines of the file:
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@@
     (stroke (width 0) (type default))
+  )
+  (rectangle (start 60.96 22.86) (end 162.56 71.12)
+    (stroke (width 0) (type default))
+    (fill (type none))
   )
   (text "PIN mappings was carefully designed to supporrt\nthe both DE0 and DE1 GPIO connector. \nDE0 board has 2xCLK_IN (1,3) and 2xCLK_OUT (19,21) pins,\nwhich are not present on DE1. These pins cannot operate\nas bi-directional IO signals, and therefore they were \nassigned to specific functions in teh interface - the direction of \ntheir signals must not be changed.\n"
@@
     (effects (font (size 1.27 1.27)) (justify left bottom))
   )
+  (text "v2.0 Bug: CS2 & RFSH sharing same pin but  OE is grounded.\nRFSH should not be wired (soldered) in U4 to avoid issues."
+    (at 88.9 27.94 0)
+    (effects (font (size 1 1)) (justify left bottom))
+  )
   (global_label "Vdd" (shape input) (at 83.439 118.364 0) (fields_autoplaced)

Commit message: V2.01
Parts:
- added J5: RFSH_CS2, Jumper:SolderJumper-3_P1.3mm_Open_RoundedPad1.0x1.5mm, symbol Connector:Conn_01x03_Female
Connections:
- net /C_CS2_RFSH: now also J5.2 (Pin_2); no longer U4.16 (B3), U5.14 (B5)
- new net /C_CS2: J5.3 (Pin_3), U5.14 (B5)
- new net /C_RFSH: J5.1 (Pin_1), U4.16 (B3)
Other:
- moved on the sheet: RN1
Changed lines of the file:
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@@
   (title_block
     (title "MSX FPGA Hat")
-    (date "2023-12-18")
-    (rev "2.0")
+    (date "2024-02-03")
+    (rev "2.01")
     (company "RCC @ 2024")
     (comment 1 "to 3.3v systems with voltage conversion")
@@
     )
   )
-  (global_label "Vcc" (shape input) (at 162.56 151.13 0) (fields_autoplaced)
-    (effects (font (size 1.27 1.27)) (justify left))
-    (property "Intersheetrefs" "${INTERSHEET_REFS}" (at 167.4816 151.13 0)
+  (global_label "Vcc" (shape input) (at 141.0155 146.1254 0) (fields_autoplaced)
+    (effects (font (size 1.27 1.27)) (justify left))
+    (property "Intersheetrefs" "${INTERSHEET_REFS}" (at 145.9371 146.1254 0)
       (effects (font (size 1.27 1.27)) (justify left) hide)
     )
@@
     )
   )
+  (global_label "{slash}C_CS2_RFSH" (shape output) (at 167.64 154.94 180) (fields_autoplaced)
+    (effects (font (size 1.27 1.27)) (justify right))
+    (property "Intersheetrefs" "${INTERSHEET_REFS}" (at 151.5315 154.94 0)
+      (effects (font (size 1.27 1.27)) (justify right) hide)
+    )
+  )
   (global_label "Vdd" (shape input) (at 73.025 80.899 180) (fields_autoplaced)
     (effects (font (size 1.27 1.27)) (justify right))
@@
     )
   )
-  (global_label "D2" (shape input) (at 152.4 156.21 180) (fields_autoplaced)
-    (effects (font (size 1.27 1.27)) (justify right))
-    (property "Intersheetrefs" "${INTERSHEET_REFS}" (at 146.9353 156.21 0)
+  (global_label "D2" (shape input) (at 130.8555 151.2054 180) (fields_autoplaced)
+    (effects (font (size 1.27 1.27)) (justify right))
+    (property "Intersheetrefs" "${INTERSHEET_REFS}" (at 125.3908 151.2054 0)
       (effects (font (size 1.27 1.27)) (justify right) hide)
     )
@@
     )
   )
-  (global_label "{slash}C_CS2_RFSH" (shape output) (at 90.297 47.879 0) (fields_autoplaced)
-    (effects (font (size 1.27 1.27)) (justify left))
-    (property "Intersheetrefs" "${INTERSHEET_REFS}" (at 106.4055 47.879 0)
+  (global_label "{slash}C_RFSH" (shape output) (at 90.297 47.879 0) (fields_autoplaced)
+    (effects (font (size 1.27 1.27)) (justify left))
+    (property "Intersheetrefs" "${INTERSHEET_REFS}" (at 101.7489 47.879 0)
       (effects (font (size 1.27 1.27)) (justify left) hide)
     )
@@
     )
   )
-  (global_label "D5" (shape input) (at 152.4 163.83 180) (fields_autoplaced)
-    (effects (font (size 1.27 1.27)) (justify right))
-    (property "Intersheetrefs" "${INTERSHEET_REFS}" (at 146.9353 163.83 0)
+  (global_label "D5" (shape input) (at 130.8555 158.8254 180) (fields_autoplaced)
+    (effects (font (size 1.27 1.27)) (justify right))
+    (property "Intersheetrefs" "${INTERSHEET_REFS}" (at 125.3908 158.8254 0)
       (effects (font (size 1.27 1.27)) (justify right) hide)
     )
@@
     )
   )
+  (global_label "{slash}C_RFSH" (shape input) (at 167.64 152.4 180) (fields_autoplaced)
+    (effects (font (size 1.27 1.27)) (justify right))
+    (property "Intersheetrefs" "${INTERSHEET_REFS}" (at 156.1881 152.4 0)
+      (effects (font (size 1.27 1.27)) (justify right) hide)
+    )
+  )
   (global_label "Vdd" (shape input) (at 33.0304 276.86 180) (fields_autoplaced)
     (effects (font (size 1.27 1.27)) (justify right))
@@
     )
   )
-  (global_label "D0" (shape input) (at 152.4 151.13 180) (fields_autoplaced)
-    (effects (font (size 1.27 1.27)) (justify right))
-    (property "Intersheetrefs" "${INTERSHEET_REFS}" (at 146.9353 151.13 0)
+  (global_label "D0" (shape input) (at 130.8555 146.1254 180) (fields_autoplaced)
+    (effects (font (size 1.27 1.27)) (justify right))
+    (property "Intersheetrefs" "${INTERSHEET_REFS}" (at 125.3908 146.1254 0)
       (effects (font (size 1.27 1.27)) (justify right) hide)
     )
@@
     )
   )
-  (global_label "{slash}C_CS2_RFSH" (shape output) (at 144.145 52.705 0) (fields_autoplaced)
-    (effects (font (size 1.27 1.27)) (justify left))
-    (property "Intersheetrefs" "${INTERSHEET_REFS}" (at 160.2535 52.705 0)
+  (global_label "{slash}C_CS2" (shape output) (at 144.145 52.705 0) (fields_autoplaced)
+    (effects (font (size 1.27 1.27)) (justify left))
+    (property "Intersheetrefs" "${INTERSHEET_REFS}" (at 154.3873 52.705 0)
       (effects (font (size 1.27 1.27)) (justify left) hide)
     )
@@
     )
   )
-  (global_label "D3" (shape input) (at 152.4 158.75 180) (fields_autoplaced)
-    (effects (font (size 1.27 1.27)) (justify right))
-    (property "Intersheetrefs" "${INTERSHEET_REFS}" (at 146.9353 158.75 0)
+  (global_label "D3" (shape input) (at 130.8555 153.7454 180) (fields_autoplaced)
+    (effects (font (size 1.27 1.27)) (justify right))
+    (property "Intersheetrefs" "${INTERSHEET_REFS}" (at 125.3908 153.7454 0)
       (effects (font (size 1.27 1.27)) (justify right) hide)
     )
@@
     )
   )
-  (global_label "D7" (shape input) (at 152.4 168.91 180) (fields_autoplaced)
-    (effects (font (size 1.27 1.27)) (justify right))
-    (property "Intersheetrefs" "${INTERSHEET_REFS}" (at 146.9353 168.91 0)
+  (global_label "D7" (shape input) (at 130.8555 163.9054 180) (fields_autoplaced)
+    (effects (font (size 1.27 1.27)) (justify right))
+    (property "Intersheetrefs" "${INTERSHEET_REFS}" (at 125.3908 163.9054 0)
       (effects (font (size 1.27 1.27)) (justify right) hide)
     )
@@
     )
   )
-  (global_label "D1" (shape input) (at 152.4 153.67 180) (fields_autoplaced)
-    (effects (font (size 1.27 1.27)) (justify right))
-    (property "Intersheetrefs" "${INTERSHEET_REFS}" (at 146.9353 153.67 0)
+  (global_label "D1" (shape input) (at 130.8555 148.6654 180) (fields_autoplaced)
+    (effects (font (size 1.27 1.27)) (justify right))
+    (property "Intersheetrefs" "${INTERSHEET_REFS}" (at 125.3908 148.6654 0)
       (effects (font (size 1.27 1.27)) (justify right) hide)
     )
@@
     )
   )
-  (global_label "D4" (shape input) (at 152.4 161.29 180) (fields_autoplaced)
-    (effects (font (size 1.27 1.27)) (justify right))
-    (property "Intersheetrefs" "${INTERSHEET_REFS}" (at 146.9353 161.29 0)
+  (global_label "D4" (shape input) (at 130.8555 156.2854 180) (fields_autoplaced)
+    (effects (font (size 1.27 1.27)) (justify right))
+    (property "Intersheetrefs" "${INTERSHEET_REFS}" (at 125.3908 156.2854 0)
       (effects (font (size 1.27 1.27)) (justify right) hide)
     )
@@
     )
   )
-  (global_label "D6" (shape input) (at 152.4 166.37 180) (fields_autoplaced)
-    (effects (font (size 1.27 1.27)) (justify right))
-    (property "Intersheetrefs" "${INTERSHEET_REFS}" (at 146.9353 166.37 0)
+  (global_label "D6" (shape input) (at 130.8555 161.3654 180) (fields_autoplaced)
+    (effects (font (size 1.27 1.27)) (justify right))
+    (property "Intersheetrefs" "${INTERSHEET_REFS}" (at 125.3908 161.3654 0)
       (effects (font (size 1.27 1.27)) (justify right) hide)
     )
@@
     (property "Intersheetrefs" "${INTERSHEET_REFS}" (at 77.47 205.2634 90)
       (effects (font (size 1.27 1.27)) (justify left) hide)
+    )
+  )
+  (global_label "{slash}C_CS2" (shape input) (at 167.64 157.48 180) (fields_autoplaced)
+    (effects (font (size 1.27 1.27)) (justify right))
+    (property "Intersheetrefs" "${INTERSHEET_REFS}" (at 157.3977 157.48 0)
+      (effects (font (size 1.27 1.27)) (justify right) hide)
     )
   )
@@
         (path "/aac9604b-8c84-42de-bd09-e07036aaaac8"
           (reference "J2") (unit 1)
+        )
+      )
+    )
+  )
+  (symbol (lib_id "Connector:Conn_01x03_Female") (at 172.72 154.94 0) (unit 1)
+    (in_bom yes) (on_board yes) (dnp no) (fields_autoplaced)
+    (property "Reference" "J5" (at 173.99 153.6699 0)
+      (effects (font (size 1.27 1.27)) (justify left))
+    )
+    (property "Value" "RFSH_CS2" (at 173.99 156.2099 0)
+      (effects (font (size 1.27 1.27)) (justify left))
+    )
+    (property "Footprint" "Jumper:SolderJumper-3_P1.3mm_Open_RoundedPad1.0x1.5mm" (at 172.72 154.94 0)
+      (effects (font (size 1.27 1.27)) hide)
+    )
+    (property "Datasheet" "~" (at 172.72 154.94 0)
+      (effects (font (size 1.27 1.27)) hide)
+    )
+    (pin "1")
+    (pin "2")
+    (pin "3")
+    (instances
+      (project "MSX_FPGA_Hat"
+        (path "/60e41f87-a5cd-4c0a-8c83-80ed9a1ad976"
+          (reference "J5") (unit 1)
         )
       )
@@
     )
   )
-  (symbol (lib_id "Device:R_Network08_US") (at 157.48 161.29 270) (unit 1)
+  (symbol (lib_id "Device:R_Network08_US") (at 135.9355 156.2854 270) (unit 1)
     (in_bom yes) (on_board yes) (dnp no)
-    (property "Reference" "RN1" (at 157.48 146.685 90)
+    (property "Reference" "RN1" (at 135.9355 141.6804 90)
       (effects (font (size 1.27 1.27)))
     )
-    (property "Value" "10K" (at 157.48 148.59 90)
+    (property "Value" "10K" (at 135.9355 143.5854 90)
       (effects (font (size 1.27 1.27)))
     )
-    (property "Footprint" "Resistor_THT:R_Array_SIP9" (at 157.48 173.355 90)
-      (effects (font (size 1.27 1.27)) hide)
-    )
-    (property "Datasheet" "http://www.vishay.com/docs/31509/csc.pdf" (at 157.48 161.29 0)
-      (effects (font (size 1.27 1.27)) hide)
-    )
+    (property "Footprint" "Resistor_THT:R_Array_SIP9" (at 135.9355 168.3504 90)
+      (effects (font (size 1.27 1.27)) hide)
+    )
+    (property "Datasheet" "http://www.vishay.com/docs/31509/csc.pdf" (at 135.9355 156.2854 0)
+      (effects (font (size 1.27 1.27)) hide)
+    )

Commit message: Master is currentl under development and tests for v2.0
Parts:
- removed J5: RFSH_CS2, Jumper:SolderJumper-3_P1.3mm_Open_RoundedPad1.0x1.5mm, symbol Connector:Conn_01x03_Female
Connections:
- net /C_CS2_RFSH is gone; now on net /C_RFSH: IDC1.6 (Pin_6)
- net GNDREF: now also U4.19 (/OE)
- net /C_CS2: now also IDC1.10 (Pin_10)
- removed net /C_U4_OE: IDC1.10 (Pin_10), U4.19 (/OE)
Changed lines of the file:
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@@
-    )
-  )
-  (global_label "{slash}C_CS2_RFSH" (shape output) (at 167.64 154.94 180) (fields_autoplaced)
-    (effects (font (size 1.27 1.27)) (justify right))
-    (property "Intersheetrefs" "${INTERSHEET_REFS}" (at 151.5315 154.94 0)
-      (effects (font (size 1.27 1.27)) (justify right) hide)
     )
   )
@@
     )
   )
+  (global_label "{slash}C_RFSH" (shape input) (at 160.3734 86.995 0) (fields_autoplaced)
+    (effects (font (size 1.27 1.27)) (justify left))
+    (property "Intersheetrefs" "${INTERSHEET_REFS}" (at 171.8253 86.995 0)
+      (effects (font (size 1.27 1.27)) (justify left) hide)
+    )
+  )
   (global_label "MSX_3.3V" (shape input) (at 86.995 247.65 0) (fields_autoplaced)
     (effects (font (size 1.27 1.27)) (justify left))
@@
     )
   )
-  (global_label "{slash}C_RFSH" (shape input) (at 167.64 152.4 180) (fields_autoplaced)
-    (effects (font (size 1.27 1.27)) (justify right))
-    (property "Intersheetrefs" "${INTERSHEET_REFS}" (at 156.1881 152.4 0)
-      (effects (font (size 1.27 1.27)) (justify right) hide)
-    )
-  )
   (global_label "Vdd" (shape input) (at 33.0304 276.86 180) (fields_autoplaced)
     (effects (font (size 1.27 1.27)) (justify right))
@@
     )
   )
-  (global_label "{slash}C_U4_OE" (shape input) (at 90.424 37.973 0) (fields_autoplaced)
-    (effects (font (size 1.27 1.27)) (justify left))
-    (property "Intersheetrefs" "${INTERSHEET_REFS}" (at 102.9644 37.973 0)
-      (effects (font (size 1.27 1.27)) (justify left) hide)
-    )
-  )
   (global_label "A8" (shape output) (at 30.353 116.205 0) (fields_autoplaced)
     (effects (font (size 1.27 1.27)) (justify left))
@@
     )
   )
+  (global_label "{slash}C_CS2" (shape input) (at 160.3734 92.075 0) (fields_autoplaced)
+    (effects (font (size 1.27 1.27)) (justify left))
+    (property "Intersheetrefs" "${INTERSHEET_REFS}" (at 170.6157 92.075 0)
+      (effects (font (size 1.27 1.27)) (justify left) hide)
+    )
+  )
   (global_label "D1" (shape input) (at 130.8555 148.6654 180) (fields_autoplaced)
     (effects (font (size 1.27 1.27)) (justify right))
@@
     )
   )
-  (global_label "{slash}C_CS2_RFSH" (shape output) (at 160.3734 86.995 0) (fields_autoplaced)
-    (effects (font (size 1.27 1.27)) (justify left))
-    (property "Intersheetrefs" "${INTERSHEET_REFS}" (at 176.4819 86.995 0)
-      (effects (font (size 1.27 1.27)) (justify left) hide)
-    )
-  )
   (global_label "{slash}C_WR" (shape output) (at 144.145 45.085 0) (fields_autoplaced)
     (effects (font (size 1.27 1.27)) (justify left))
@@
     )
   )
-  (global_label "{slash}C_U4_OE" (shape output) (at 160.3734 92.075 0) (fields_autoplaced)
-    (effects (font (size 1.27 1.27)) (justify left))
-    (property "Intersheetrefs" "${INTERSHEET_REFS}" (at 172.9138 92.075 0)
-      (effects (font (size 1.27 1.27)) (justify left) hide)
-    )
-  )
   (global_label "Vdd" (shape input) (at 127 37.719 180) (fields_autoplaced)
     (effects (font (size 1.27 1.27)) (justify right))
@@
     (property "Intersheetrefs" "${INTERSHEET_REFS}" (at 77.47 205.2634 90)
       (effects (font (size 1.27 1.27)) (justify left) hide)
-    )
-  )
-  (global_label "{slash}C_CS2" (shape input) (at 167.64 157.48 180) (fields_autoplaced)
-    (effects (font (size 1.27 1.27)) (justify right))
-    (property "Intersheetrefs" "${INTERSHEET_REFS}" (at 157.3977 157.48 0)
-      (effects (font (size 1.27 1.27)) (justify right) hide)
     )
   )
@@
         (path "/aac9604b-8c84-42de-bd09-e07036aaaac8"
           (reference "J2") (unit 1)
-        )
-      )
-    )
-  )
-  (symbol (lib_id "Connector:Conn_01x03_Female") (at 172.72 154.94 0) (unit 1)
-    (in_bom yes) (on_board yes) (dnp no) (fields_autoplaced)
-    (property "Reference" "J5" (at 173.99 153.6699 0)
-      (effects (font (size 1.27 1.27)) (justify left))
-    )
-    (property "Value" "RFSH_CS2" (at 173.99 156.2099 0)
-      (effects (font (size 1.27 1.27)) (justify left))
-    )
-    (property "Footprint" "Jumper:SolderJumper-3_P1.3mm_Open_RoundedPad1.0x1.5mm" (at 172.72 154.94 0)
-      (effects (font (size 1.27 1.27)) hide)
-    )
-    (property "Datasheet" "~" (at 172.72 154.94 0)
-      (effects (font (size 1.27 1.27)) hide)
-    )
-    (pin "1")
-    (pin "2")
-    (pin "3")
-    (instances
-      (project "MSX_FPGA_Hat"
-        (path "/60e41f87-a5cd-4c0a-8c83-80ed9a1ad976"
-          (reference "J5") (unit 1)
         )
       )
@@
         )
       )
+    )
+  )
+  (symbol (lib_id "power:GNDREF") (at 90.424 37.973 0) (unit 1)
+    (in_bom yes) (on_board yes) (dnp no) (fields_autoplaced)
+    (property "Reference" "#PWR017" (at 90.424 44.323 0)
+      (effects (font (size 1.27 1.27)) hide)
+    )
+    (property "Value" "GNDREF" (at 90.424 43.5658 0)
+      (effects (font (size 1.27 1.27)) hide)
+    )
+    (property "Footprint" "" (at 90.424 37.973 0)
+      (effects (font (size 1.27 1.27)) hide)
+    )
+    (property "Datasheet" "" (at 90.424 37.973 0)
+      (effects (font (size 1.27 1.27)) hide)
+    )
+    (pin "1")
+    (instances
+      (project "MSX_FPGA_Hat"
+        (path "/60e41f87-a5cd-4c0a-8c83-80ed9a1ad976"
+          (reference "#PWR017") (unit 1)
+        )
+      )
